Commit message: xe 4 banh

File: src/waiter_description/urdf/waiter.xacro (robot description, xacro)
@@ -8,7 +8,7 @@
   <xacro:property name="wheel_width" value="0.045"/>
   <xacro:property name="wheel_mass" value="1.2"/>
+  <xacro:property name="wheel_front_x_offset" value="0.14"/>
+  <xacro:property name="wheel_rear_x_offset" value="-0.14"/>
   <xacro:property name="wheel_y_offset" value="0.245"/>
-  <xacro:property name="caster_radius" value="0.035"/>
-  <xacro:property name="caster_mass" value="0.35"/>
   <xacro:property name="lidar_radius" value="0.05"/>
   <xacro:property name="lidar_height" value="0.06"/>
@@ -38,4 +38,30 @@
     </inertial>
   </xacro:macro>
+  <xacro:macro name="drive_wheel" params="prefix x y">
+    <link name="${prefix}_wheel_link">
+      <visual>
+        <origin xyz="0 0 0" rpy="1.5708 0 0"/>
+        <geometry>
+          <cylinder radius="${wheel_radius}" length="${wheel_width}"/>
+        </geometry>
+        <material name="wheel_black">
+          <color rgba="0.08 0.08 0.08 1.0"/>
+        </material>
+      </visual>
+      <collision>
+        <origin xyz="0 0 0" rpy="1.5708 0 0"/>
+        <geometry>
+          <cylinder radius="${wheel_radius}" length="${wheel_width}"/>
+        </geometry>
+      </collision>
+      <xacro:inertial_cylinder mass="${wheel_mass}" radius="${wheel_radius}" length="${wheel_width}"/>
+    </link>
+    <joint name="${prefix}_wheel_joint" type="continuous">
+      <parent link="base_link"/>
+      <child link="${prefix}_wheel_link"/>
+      <origin xyz="${x} ${y} ${wheel_radius}" rpy="0 0 0"/>
+      <axis xyz="0 1 0"/>
+    </joint>
+  </xacro:macro>
   <link name="base_link">
     <visual>
@@ -56,73 +82,8 @@
     <xacro:inertial_cylinder mass="${base_mass}" radius="${base_radius}" length="${base_height}"/>
   </link>
-  <link name="left_wheel_link">
-    <visual>
-      <origin xyz="0 0 0" rpy="1.5708 0 0"/>
-      <geometry>
-        <cylinder radius="${wheel_radius}" length="${wheel_width}"/>
-      </geometry>
-      <material name="wheel_black">
-        <color rgba="0.08 0.08 0.08 1.0"/>
-      </material>
-    </visual>
-    <collision>
-      <origin xyz="0 0 0" rpy="1.5708 0 0"/>
-      <geometry>
-        <cylinder radius="${wheel_radius}" length="${wheel_width}"/>
-      </geometry>
-    </collision>
-    <xacro:inertial_cylinder mass="${wheel_mass}" radius="${wheel_radius}" length="${wheel_width}"/>
-  </link>
-  <joint name="left_wheel_joint" type="continuous">
-    <parent link="base_link"/>
-    <child link="left_wheel_link"/>
-    <origin xyz="0 ${wheel_y_offset} ${wheel_radius}" rpy="0 0 0"/>
-    <axis xyz="0 1 0"/>
-  </joint>
-  <link name="right_wheel_link">
-    <visual>
-      <origin xyz="0 0 0" rpy="1.5708 0 0"/>
-      <geometry>
-        <cylinder radius="${wheel_radius}" length="${wheel_width}"/>
-      </geometry>
-      <material name="wheel_black"/>
-    </visual>
-    <collision>
-      <origin xyz="0 0 0" rpy="1.5708 0 0"/>
-      <geometry>
-        <cylinder radius="${wheel_radius}" length="${wheel_width}"/>
-      </geometry>
-    </collision>
-    <xacro:inertial_cylinder mass="${wheel_mass}" radius="${wheel_radius}" length="${wheel_width}"/>
-  </link>
-  <joint name="right_wheel_joint" type="continuous">
-    <parent link="base_link"/>
-    <child link="right_wheel_link"/>
-    <origin xyz="0 -${wheel_y_offset} ${wheel_radius}" rpy="0 0 0"/>
-    <axis xyz="0 1 0"/>
-  </joint>
-  <link name="caster_link">
-    <visual>
-      <origin xyz="0 0 0" rpy="0 0 0"/>
-      <geometry>
-        <sphere radius="${caster_radius}"/>
-      </geometry>
-      <material name="caster_silver">
-        <color rgba="0.75 0.75 0.78 1.0"/>
-      </material>
-    </visual>
-    <collision>
-      <origin xyz="0 0 0" rpy="0 0 0"/>
-      <geometry>
-        <sphere radius="${caster_radius}"/>
-      </geometry>
-    </collision>
-    <xacro:inertial_sphere mass="${caster_mass}" radius="${caster_radius}"/>
-  </link>
-  <joint name="caster_joint" type="fixed">
-    <parent link="base_link"/>
-    <child link="caster_link"/>
-    <origin xyz="-${base_radius * 0.70} 0 ${caster_radius}" rpy="0 0 0"/>
-  </joint>
+  <xacro:drive_wheel prefix="front_left" x="${wheel_front_x_offset}" y="${wheel_y_offset}"/>
+  <xacro:drive_wheel prefix="rear_left" x="${wheel_rear_x_offset}" y="${wheel_y_offset}"/>
+  <xacro:drive_wheel prefix="front_right" x="${wheel_front_x_offset}" y="-${wheel_y_offset}"/>
+  <xacro:drive_wheel prefix="rear_right" x="${wheel_rear_x_offset}" y="-${wheel_y_offset}"/>
   <link name="lidar_link">
     <visual>
@@ -226,24 +187,31 @@
   </joint>
   <!-- Wheel-ground friction and contact tuning for stable turns in Gazebo -->
-  <gazebo reference="left_wheel_link">
-    <mu1>1.2</mu1>
-    <mu2>1.2</mu2>
-    <kp>1000000.0</kp>
-    <kd>10.0</kd>
-    <material>Gazebo/Black</material>
-  </gazebo>
-  <gazebo reference="right_wheel_link">
-    <mu1>1.2</mu1>
-    <mu2>1.2</mu2>
-    <kp>1000000.0</kp>
-    <kd>10.0</kd>
-    <material>Gazebo/Black</material>
-  </gazebo>
-  <gazebo reference="caster_link">
-    <mu1>0.2</mu1>
-    <mu2>0.2</mu2>
-    <kp>1000000.0</kp>
-    <kd>1.0</kd>
-    <material>Gazebo/Grey</material>
+  <gazebo reference="front_left_wheel_link">
+    <mu1>1.2</mu1>
+    <mu2>1.2</mu2>
+    <kp>1000000.0</kp>
+    <kd>10.0</kd>
+    <material>Gazebo/Black</material>
+  </gazebo>
+  <gazebo reference="rear_left_wheel_link">
+    <mu1>1.2</mu1>
+    <mu2>1.2</mu2>
+    <kp>1000000.0</kp>
+    <kd>10.0</kd>
+    <material>Gazebo/Black</material>
+  </gazebo>
+  <gazebo reference="front_right_wheel_link">
+    <mu1>1.2</mu1>
+    <mu2>1.2</mu2>
+    <kp>1000000.0</kp>
+    <kd>10.0</kd>
+    <material>Gazebo/Black</material>
+  </gazebo>
+  <gazebo reference="rear_right_wheel_link">
+    <mu1>1.2</mu1>
+    <mu2>1.2</mu2>
+    <kp>1000000.0</kp>
+    <kd>10.0</kd>
+    <material>Gazebo/Black</material>
   </gazebo>
   <gazebo reference="lidar_link">
@@ -253,6 +221,8 @@
     <plugin filename="gz-sim-joint-state-publisher-system" name="gz::sim::systems::JointStatePublisher"/>
     <plugin filename="gz-sim-diff-drive-system" name="gz::sim::systems::DiffDrive">
-      <left_joint>left_wheel_joint</left_joint>
-      <right_joint>right_wheel_joint</right_joint>
+      <left_joint>front_left_wheel_joint</left_joint>
+      <left_joint>rear_left_wheel_joint</left_joint>
+      <right_joint>front_right_wheel_joint</right_joint>
+      <right_joint>rear_right_wheel_joint</right_joint>
       <wheel_separation>${2.0 * wheel_y_offset}</wheel_separation>
       <wheel_radius>${wheel_radius}</wheel_radius>
@@ -262,6 +232,6 @@
       <frame_id>odom</frame_id>
       <child_frame_id>base_link</child_frame_id>
-      <max_linear_acceleration>1.0</max_linear_acceleration>
-      <max_angular_acceleration>2.0</max_angular_acceleration>
+      <max_linear_acceleration>0.55</max_linear_acceleration>
+      <max_angular_acceleration>1.1</max_angular_acceleration>
     </plugin>
   </gazebo>

Commit message: feat: new robot shape

File: src/waiter_description/urdf/waiter.xacro (robot description, xacro)
@@ -1,223 +1,147 @@
 <?xml version="1.0"?>
+<!-- ================================================================
+  Waiter Robot URDF – Multi-part service robot design
+  - Base platform (wide, low) with 4 wheels
+  - Central column/pillar
+  - Serving tray at table height (~0.72 m)
+  - 2D LiDAR on top
+================================================================ -->
 <robot xmlns:xacro="http://www.ros.org/wiki/xacro" name="waiter_robot">
-  <!-- Robot dimensions -->
-  <xacro:property name="base_radius" value="0.23"/>
-  <xacro:property name="base_height" value="0.28"/>
-  <xacro:property name="base_mass" value="22.0"/>
-  <xacro:property name="wheel_radius" value="0.08"/>
-  <xacro:property name="wheel_width" value="0.045"/>
-  <xacro:property name="wheel_mass" value="1.2"/>
-  <xacro:property name="wheel_front_x_offset" value="0.14"/>
-  <xacro:property name="wheel_rear_x_offset" value="-0.14"/>
-  <xacro:property name="wheel_y_offset" value="0.245"/>
-  <xacro:property name="lidar_radius" value="0.05"/>
-  <xacro:property name="lidar_height" value="0.06"/>
-  <xacro:property name="lidar_mass" value="0.25"/>
-  <xacro:macro name="inertial_cylinder" params="mass radius length">
+  <!-- ===================== PROPERTIES ===================== -->
+  <!-- Wheels -->
+  <xacro:property name="wheel_radius" value="0.05"/>
+  <xacro:property name="wheel_width"  value="0.03"/>
+  <xacro:property name="wheel_mass"   value="0.5"/>
+  <xacro:property name="wheel_x"      value="0.13"/>
+  <xacro:property name="wheel_y"      value="0.19"/>
+  <!-- Base platform (where wheels attach) -->
+  <xacro:property name="base_radius"  value="0.22"/>
+  <xacro:property name="base_height"  value="0.06"/>
+  <xacro:property name="base_mass"    value="8.0"/>
+  <!-- Central column -->
+  <xacro:property name="col_radius"   value="0.06"/>
+  <xacro:property name="col_height"   value="0.58"/>
+  <xacro:property name="col_mass"     value="3.0"/>
+  <!-- Serving tray -->
+  <xacro:property name="tray_radius"  value="0.18"/>
+  <xacro:property name="tray_height"  value="0.025"/>
+  <xacro:property name="tray_mass"    value="1.0"/>
+  <!-- LiDAR -->
+  <xacro:property name="lidar_radius" value="0.035"/>
+  <xacro:property name="lidar_height" value="0.03"/>
+  <!-- ===================== MACROS ========================= -->
+  <xacro:macro name="cylinder_inertia" params="m r h">
     <inertial>
-      <mass value="${mass}"/>
-      <origin xyz="0 0 0" rpy="0 0 0"/>
-      <inertia ixx="${(1.0/12.0) * mass * (3.0 * radius * radius + length * length)}"
-               ixy="0.0"
-               ixz="0.0"
-               iyy="${(1.0/12.0) * mass * (3.0 * radius * radius + length * length)}"
-               iyz="0.0"
-               izz="${0.5 * mass * radius * radius}"/>
+      <mass value="${m}"/>
+      <inertia ixx="${(1.0/12.0)*m*(3*r*r + h*h)}" ixy="0" ixz="0"
+               iyy="${(1.0/12.0)*m*(3*r*r + h*h)}" iyz="0"
+               izz="${0.5*m*r*r}"/>
     </inertial>
   </xacro:macro>
-  <xacro:macro name="inertial_sphere" params="mass radius">
-    <inertial>
-      <mass value="${mass}"/>
-      <origin xyz="0 0 0" rpy="0 0 0"/>
-      <inertia ixx="${0.4 * mass * radius * radius}"
-               ixy="0.0"
-               ixz="0.0"
-               iyy="${0.4 * mass * radius * radius}"
-               iyz="0.0"
-               izz="${0.4 * mass * radius * radius}"/>
-    </inertial>
-  </xacro:macro>
-  <xacro:macro name="drive_wheel" params="prefix x y">
+  <!-- Wheel macro -->
+  <xacro:macro name="wheel" params="prefix x_pos y_pos">
     <link name="${prefix}_wheel_link">
       <visual>
-        <origin xyz="0 0 0" rpy="1.5708 0 0"/>
-        <geometry>
-          <cylinder radius="${wheel_radius}" length="${wheel_width}"/>
-        </geometry>
-        <material name="wheel_black">
-          <color rgba="0.08 0.08 0.08 1.0"/>
-        </material>
+        <geometry><cylinder radius="${wheel_radius}" length="${wheel_width}"/></geometry>
+        <material name="dark_grey"><color rgba="0.15 0.15 0.15 1"/></material>
       </visual>
       <collision>
-        <origin xyz="0 0 0" rpy="1.5708 0 0"/>
-        <geometry>
-          <cylinder radius="${wheel_radius}" length="${wheel_width}"/>
-        </geometry>
+        <geometry><cylinder radius="${wheel_radius}" length="${wheel_width}"/></geometry>
+        <surface>
+          <friction>
+            <ode><mu>1.0</mu><mu2>1.0</mu2></ode>
+          </friction>
+        </surface>
       </collision>
-      <xacro:inertial_cylinder mass="${wheel_mass}" radius="${wheel_radius}" length="${wheel_width}"/>
+      <xacro:cylinder_inertia m="${wheel_mass}" r="${wheel_radius}" h="${wheel_width}"/>
     </link>
     <joint name="${prefix}_wheel_joint" type="continuous">
       <parent link="base_link"/>
-      <child link="${prefix}_wheel_link"/>
-      <origin xyz="${x} ${y} ${wheel_radius}" rpy="0 0 0"/>
-      <axis xyz="0 1 0"/>
+      <child  link="${prefix}_wheel_link"/>
+      <!-- Wheels at axle height (z=0 in base_link frame = wheel_radius above ground) -->
+      <origin xyz="${x_pos} ${y_pos} 0" rpy="${-pi/2} 0 0"/>
+      <axis xyz="0 0 1"/>
+      <dynamics damping="0.01" friction="0.1"/>
     </joint>
   </xacro:macro>
+  <!-- ===================== LINKS ========================== -->
+  <!-- Ground-level reference -->
+  <link name="base_footprint"/>
+  <!-- Base platform – wide flat disk at wheel axle height -->
   <link name="base_link">
     <visual>
-      <origin xyz="0 0 ${wheel_radius + base_height / 2.0}" rpy="0 0 0"/>
-      <geometry>
-        <cylinder radius="${base_radius}" length="${base_height}"/>
-      </geometry>
-      <material name="body_gray">
-        <color rgba="0.25 0.25 0.28 1.0"/>
-      </material>
+      <geometry><cylinder radius="${base_radius}" length="${base_height}"/></geometry>
+      <material name="charcoal"><color rgba="0.25 0.25 0.28 1"/></material>
     </visual>
     <collision>
-      <origin xyz="0 0 ${wheel_radius + base_height / 2.0}" rpy="0 0 0"/>
-      <geometry>
-        <cylinder radius="${base_radius}" length="${base_height}"/>
-      </geometry>
+      <geometry><cylinder radius="${base_radius}" length="${base_height}"/></geometry>
     </collision>
-    <xacro:inertial_cylinder mass="${base_mass}" radius="${base_radius}" length="${base_height}"/>
+    <xacro:cylinder_inertia m="${base_mass}" r="${base_radius}" h="${base_height}"/>
   </link>
-  <xacro:drive_wheel prefix="front_left" x="${wheel_front_x_offset}" y="${wheel_y_offset}"/>
-  <xacro:drive_wheel prefix="rear_left" x="${wheel_rear_x_offset}" y="${wheel_y_offset}"/>
-  <xacro:drive_wheel prefix="front_right" x="${wheel_front_x_offset}" y="-${wheel_y_offset}"/>
-  <xacro:drive_wheel prefix="rear_right" x="${wheel_rear_x_offset}" y="-${wheel_y_offset}"/>
+  <!-- base_footprint → base_link: lift so wheel bottoms touch ground -->
+  <joint name="base_joint" type="fixed">
+    <parent link="base_footprint"/>
+    <child  link="base_link"/>
+    <origin xyz="0 0 ${wheel_radius}" rpy="0 0 0"/>
+  </joint>
+  <!-- Central column/pillar -->
+  <link name="column_link">
+    <visual>
+      <geometry><cylinder radius="${col_radius}" length="${col_height}"/></geometry>
+      <material name="silver"><color rgba="0.7 0.7 0.72 1"/></material>
+    </visual>
+    <collision>
+      <geometry><cylinder radius="${col_radius}" length="${col_height}"/></geometry>
+    </collision>
+    <xacro:cylinder_inertia m="${col_mass}" r="${col_radius}" h="${col_height}"/>
+  </link>
+  <joint name="column_joint" type="fixed">
+    <parent link="base_link"/>
+    <child  link="column_link"/>
+    <origin xyz="0 0 ${base_height/2 + col_height/2}" rpy="0 0 0"/>
+  </joint>
+  <!-- Serving tray -->
+  <link name="tray_link">
+    <visual>
+      <geometry><cylinder radius="${tray_radius}" length="${tray_height}"/></geometry>
+      <material name="orange"><color rgba="0.9 0.5 0.1 1"/></material>
+    </visual>
+    <collision>
+      <geometry><cylinder radius="${tray_radius}" length="${tray_height}"/></geometry>
+    </collision>
+    <xacro:cylinder_inertia m="${tray_mass}" r="${tray_radius}" h="${tray_height}"/>
+  </link>
+  <joint name="tray_joint" type="fixed">
+    <parent link="column_link"/>
+    <child  link="tray_link"/>
+    <origin xyz="0 0 ${col_height/2 + tray_height/2}" rpy="0 0 0"/>
+  </joint>
+  <!-- LiDAR sensor on top of tray -->
   <link name="lidar_link">
     <visual>
-      <origin xyz="0 0 0" rpy="0 0 0"/>
-      <geometry>
-        <cylinder radius="${lidar_radius}" length="${lidar_height}"/>
-      </geometry>
-      <material name="lidar_blue">
-        <color rgba="0.1 0.45 0.75 1.0"/>
-      </material>
+      <geometry><cylinder radius="${lidar_radius}" length="${lidar_height}"/></geometry>
+      <material name="blue"><color rgba="0.1 0.1 0.8 1"/></material>
     </visual>
     <collision>
-      <origin xyz="0 0 0" rpy="0 0 0"/>
-      <geometry>
-        <cylinder radius="${lidar_radius}" length="${lidar_height}"/>
-      </geometry>
+      <geometry><cylinder radius="${lidar_radius}" length="${lidar_height}"/></geometry>
     </collision>
-    <xacro:inertial_cylinder mass="${lidar_mass}" radius="${lidar_radius}" length="${lidar_height}"/>
+    <inertial>
+      <mass value="0.1"/>
+      <inertia ixx="0.0001" ixy="0" ixz="0" iyy="0.0001" iyz="0" izz="0.0001"/>
+    </inertial>
   </link>
   <joint name="lidar_joint" type="fixed">
-    <parent link="base_link"/>
-    <child link="lidar_link"/>
-    <origin xyz="0 0 ${base_height + lidar_height / 2.0}" rpy="0 0 0"/>
+    <parent link="tray_link"/>
+    <child  link="lidar_link"/>
+    <origin xyz="0 0 ${tray_height/2 + lidar_height/2}" rpy="0 0 0"/>
   </joint>
-  <link name="torso_link">
-    <visual>
-      <origin xyz="0 0 0" rpy="0 0 0"/>
-      <geometry>
-        <cylinder radius="0.18" length="0.42"/>
-      </geometry>
-      <material name="torso_white">
-        <color rgba="0.92 0.92 0.94 1.0"/>
-      </material>
-    </visual>
-    <visual>
-      <origin xyz="0.15 0 0.0" rpy="0 0 0"/>
-      <geometry>
-        <box size="0.06 0.20 0.22"/>
-      </geometry>
-      <material name="front_screen">
-        <color rgba="0.14 0.18 0.22 1.0"/>
-      </material>
-    </visual>
-    <xacro:inertial_cylinder mass="2.8" radius="0.18" length="0.42"/>
-  </link>
-  <joint name="torso_joint" type="fixed">
-    <parent link="base_link"/>
-    <child link="torso_link"/>
-    <origin xyz="0 0 ${base_height + 0.21}" rpy="0 0 0"/>
-  </joint>
-  <link name="tray_lower_link">
-    <visual>
-      <origin xyz="0 0 0" rpy="0 0 0"/>
-      <geometry>
-        <cylinder radius="0.22" length="0.03"/>
-      </geometry>
-      <material name="tray_dark">
-        <color rgba="0.2 0.2 0.22 1.0"/>
-      </material>
-    </visual>
-    <xacro:inertial_cylinder mass="0.6" radius="0.22" length="0.03"/>
-  </link>
-  <joint name="tray_lower_joint" type="fixed">
-    <parent link="torso_link"/>
-    <child link="tray_lower_link"/>
-    <origin xyz="0 0 0.08" rpy="0 0 0"/>
-  </joint>
-  <link name="tray_upper_link">
-    <visual>
-      <origin xyz="0 0 0" rpy="0 0 0"/>
-      <geometry>
-        <cylinder radius="0.23" length="0.03"/>
-      </geometry>
-      <material name="tray_dark_2">
-        <color rgba="0.22 0.22 0.25 1.0"/>
-      </material>
-    </visual>
-    <xacro:inertial_cylinder mass="0.6" radius="0.23" length="0.03"/>
-  </link>
-  <joint name="tray_upper_joint" type="fixed">
-    <parent link="torso_link"/>
-    <child link="tray_upper_link"/>
-    <origin xyz="0 0 0.24" rpy="0 0 0"/>
-  </joint>
-  <link name="head_cap_link">
-    <visual>
-      <origin xyz="0 0 0" rpy="0 0 0"/>
-      <geometry>
-        <sphere radius="0.12"/>
-      </geometry>
-      <material name="head_white">
-        <color rgba="0.93 0.93 0.95 1.0"/>
-      </material>
-    </visual>
-    <xacro:inertial_sphere mass="0.8" radius="0.12"/>
-  </link>
-  <joint name="head_cap_joint" type="fixed">
-    <parent link="torso_link"/>
-    <child link="head_cap_link"/>
-    <origin xyz="0 0 0.31" rpy="0 0 0"/>
-  </joint>
-  <!-- Wheel-ground friction and contact tuning for stable turns in Gazebo -->
-  <gazebo reference="front_left_wheel_link">
-    <mu1>1.2</mu1>
-    <mu2>1.2</mu2>
-    <kp>1000000.0</kp>
-    <kd>10.0</kd>
-    <material>Gazebo/Black</material>
-  </gazebo>
-  <gazebo reference="rear_left_wheel_link">
-    <mu1>1.2</mu1>
-    <mu2>1.2</mu2>
-    <kp>1000000.0</kp>
-    <kd>10.0</kd>
-    <material>Gazebo/Black</material>
-  </gazebo>
-  <gazebo reference="front_right_wheel_link">
-    <mu1>1.2</mu1>
-    <mu2>1.2</mu2>
-    <kp>1000000.0</kp>
-    <kd>10.0</kd>
-    <material>Gazebo/Black</material>
-  </gazebo>
-  <gazebo reference="rear_right_wheel_link">
-    <mu1>1.2</mu1>
-    <mu2>1.2</mu2>
-    <kp>1000000.0</kp>
-    <kd>10.0</kd>
-    <material>Gazebo/Black</material>
-  </gazebo>
-  <gazebo reference="lidar_link">
-    <material>Gazebo/Blue</material>
-  </gazebo>
+  <!-- ===================== WHEELS ========================= -->
+  <xacro:wheel prefix="front_left"  x_pos="${wheel_x}"  y_pos="${wheel_y}"/>
+  <xacro:wheel prefix="front_right" x_pos="${wheel_x}"  y_pos="${-wheel_y}"/>
+  <xacro:wheel prefix="rear_left"   x_pos="${-wheel_x}" y_pos="${wheel_y}"/>
+  <xacro:wheel prefix="rear_right"  x_pos="${-wheel_x}" y_pos="${-wheel_y}"/>
+  <!-- ===================== GAZEBO PLUGINS ================= -->
+  <!-- Differential drive – 4 wheels -->
   <gazebo>
-    <plugin filename="gz-sim-joint-state-publisher-system" name="gz::sim::systems::JointStatePublisher"/>
     <plugin filename="gz-sim-diff-drive-system" name="gz::sim::systems::DiffDrive">
       <left_joint>front_left_wheel_joint</left_joint>
@@ -225,26 +149,31 @@
       <right_joint>front_right_wheel_joint</right_joint>
       <right_joint>rear_right_wheel_joint</right_joint>
-      <wheel_separation>${2.0 * wheel_y_offset}</wheel_separation>
+      <wheel_separation>${2.0 * wheel_y}</wheel_separation>
       <wheel_radius>${wheel_radius}</wheel_radius>
-      <topic>cmd_vel_nav</topic>
+      <topic>cmd_vel</topic>
       <odom_topic>odom</odom_topic>
-      <tf_topic>tf</tf_topic>
+      <!-- TF disabled – odom_tf_broadcaster handles it -->
+      <tf_topic>__unused_tf</tf_topic>
       <frame_id>odom</frame_id>
       <child_frame_id>base_link</child_frame_id>
-      <max_linear_acceleration>0.55</max_linear_acceleration>
-      <max_angular_acceleration>1.1</max_angular_acceleration>
+      <max_linear_acceleration>0.5</max_linear_acceleration>
+      <max_angular_acceleration>1.0</max_angular_acceleration>
     </plugin>
   </gazebo>
+  <!-- Joint state publisher for wheel visualization -->
+  <gazebo>
+    <plugin filename="gz-sim-joint-state-publisher-system"
+            name="gz::sim::systems::JointStatePublisher"/>
+  </gazebo>
+  <!-- 2D LiDAR sensor (360°, 6m range) -->
   <gazebo reference="lidar_link">
-    <sensor type="gpu_lidar" name="waiter_lidar_sensor">
+    <sensor name="lidar" type="gpu_lidar">
       <always_on>true</always_on>
-      <visualize>true</visualize>
-      <update_rate>12.0</update_rate>
-      <pose>0 0 0 0 0 0</pose>
+      <update_rate>10</update_rate>
       <topic>scan</topic>
-      <ray>
+      <lidar>
         <scan>
           <horizontal>
-            <samples>720</samples>
+            <samples>360</samples>
             <resolution>1</resolution>
             <min_angle>-3.14159</min_angle>
@@ -253,14 +182,9 @@
         </scan>
         <range>
-          <min>0.12</min>
-          <max>8.0</max>
+          <min>0.15</min>
+          <max>6.0</max>
           <resolution>0.01</resolution>
         </range>
-        <noise>
-          <type>gaussian</type>
-          <mean>0.0</mean>
-          <stddev>0.008</stddev>
-        </noise>
-      </ray>
+      </lidar>
     </sensor>
   </gazebo>
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